Commit message: Document Isaac Sim UR10e path planning demo

File: src/ur10e_description/urdf/ur10e.urdf (robot description, URDF)
Before this commit: robot ur10e_robot, 11 links, 10 joints
Links:
- added link end_effector, mass 0.5; collision mesh filename=package://ur10e_description/meshes/ur10e/end_effector.stl scale=0.001 0.001 0.001; visual mesh filename=package://ur10e_description/meshes/ur10e/end_effector.stl scale=0.001 0.001 0.001
- added link sim_camera
Joints:
- added joint flange-sim_camera: type fixed, parent tool0, child sim_camera, origin xyz=0 0 0 rpy=1.5707963267948966 0 1.5707963267948966
- added joint tool0-end_effector: type fixed, parent tool0, child end_effector, origin xyz=0 0 0 rpy=0 0 0
